Commit message: Update bumperbot.urdf.xacro

File: src/bumperbot_description/urdf/bumperbot.urdf.xacro (robot description, xacro)
@@ -178,5 +178,5 @@
     </link>
     <joint name="imu_joint" type="fixed">
-        <origin xyz="0 0 0.07" rpy="3.14 0 0" />
+        <origin xyz="0 0 0.07" rpy="0 0 0" />
             <parent link="base_link" />
             <child link="imu_link" />
